File: Tube AMP GU17 Power Output Stage/Tube AMP GU17 Power Output Stage.sch (KiCad schematic (older format))
At the start: 38 parts, among them J1 AIN+, J10 BRN, J11 B+, J12 BLU, J13 F, J14 FH, J15 F, J16 B+, J17 +222V, J18 VC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

Commit message: Update to a new socket
Parts:
- V1: footprint Valve:Valve_ECC-83-1 -> Tube Amp Parts:B9A-PCB-21
Changed lines of the file:
@@
 F 0 "V1" H 8750 2800 50  0000 L CNN
 F 1 "GU17" H 8750 2300 50  0000 L CNN
-F 2 "Valve:Valve_ECC-83-1" H 8650 2100 50  0001 C CNN
+F 2 "Tube Amp Parts:B9A-PCB-21" H 8650 2100 50  0001 C CNN
 F 3 "" H 8600 2550 50  0001 C CNN
 	1    8600 2550
@@
 F 0 "V1" H 1928 6463 50  0000 L CNN
 F 1 "GU17" H 1928 6372 50  0000 L CNN
-F 2 "Valve:Valve_ECC-83-1" H 1750 6050 50  0001 C CNN
+F 2 "Tube Amp Parts:B9A-PCB-21" H 1750 6050 50  0001 C CNN
 F 3 "" H 1700 6500 50  0001 C CNN
 	2    1700 6500
